Commit message: Update h2017 urdf model

File: dsr_description2/urdf/h2017.urdf (robot description, URDF)
Before this commit: robot h2017, 9 links, 8 joints
Links:
- removed link base
- link base_link: geometry collision mesh filename=package://dsr_description2/meshes/h2017_collision/H2017_0_0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 scale=0.001 0.001 0.001; visual mesh filename=package://dsr_description2/meshes/h2017_white/H2017_0_0.dae scale=0.001 0.001 0.001
- link link_1: geometry collision mesh filename=package://dsr_description2/meshes/h2017_collision/H2017_1_0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 scale=0.001 0.001 0.001; visual mesh filename=package://dsr_description2/meshes/h2017_white/H2017_1_0.dae scale=0.001 0.001 0.001
- link link_2: geometry collision mesh filename=package://dsr_description2/meshes/h2017_collision/H2017_2_0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 scale=0.001 0.001 0.001; collision mesh filename=package://dsr_description2/meshes/h2017_collision/H2017_2_1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 scale=0.001 0.001 0.001
- link link_3: geometry collision mesh filename=package://dsr_description2/meshes/h2017_collision/H2017_3_0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 scale=0.001 0.001 0.001; visual mesh filename=package://dsr_description2/meshes/h2017_white/H2017_3_0.dae scale=0.001 0.001 0.001
- link link_4: geometry collision mesh filename=package://dsr_description2/meshes/h2017_collision/H2017_4_0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 scale=0.001 0.001 0.001; collision mesh filename=package://dsr_description2/meshes/h2017_collision/H2017_4_1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 scale=0.001 0.001 0.001
- link link_5: geometry collision mesh filename=package://dsr_description2/meshes/h2017_collision/H2017_5_0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 scale=0.001 0.001 0.001; visual mesh filename=package://dsr_description2/meshes/h2017_white/H2017_5_0.dae scale=0.001 0.001 0.001
- link link_6: geometry collision mesh filename=package://dsr_description2/meshes/h2017_collision/H2017_6_0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 scale=0.001 0.001 0.001; visual mesh filename=package://dsr_description2/meshes/h2017_white/H2017_6_0.dae scale=0.001 0.001 0.001
